Commit message: add a bringup folder, include launch file

File: src/simple_delta_robot_description/urdf/delta_robot.xacro (robot description, xacro)
@@ -13,5 +13,5 @@
     <parent link="world"/>
     <child link="base_link"/>
-    <origin xyz="0 0 2" rpy="0 0 0"/>
+    <origin xyz="0 0 0.7" rpy="0 0 0"/>
   </joint>
   <link name="base_link">
